File: wearable_v1_hw/wearable_som/wearable_som.kicad_sch (KiCad schematic)
At the start: 47 parts, among them IC1 TPS7A0228PDBVR, IC2 DA7280-00FV2, J1 Conn_01x04, J2 USB4105-GF-A, J3 Conn_01x03, M1 Motor_DC, Q1 PMOS, SW1 Reset, SW2 SW_Nidec_CAS-120A1, SW3 Boot, U1 STM32WB55RGVx, U2 BMI270, U3 MCP73831-2-MC, U4 DLF162500LT-5028A1, U5 2450AT18A100E, U6 USBLC6-2SC6, Y1 Crystal_GND23, Y2 Crystal

Commit message: wearables v2
Parts:
- C11: value 100nF -> 0.1uF
- C3: value 0.1u -> 0.1uF
- C4: value 1uF -> 0.1uF
Changed lines of the file:
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@@
 			)
 		)
-		(property "Value" "0.1u"
+		(property "Value" "0.1uF"
 			(at 53.721 147.193 0)
 			(effects
@@
 			)
 		)
-		(property "Value" "1uF"
+		(property "Value" "0.1uF"
 			(at 199.39 88.8999 0)
 			(effects
@@
 		(fields_autoplaced yes)
 		(property "Reference" "C11"
-			(at 113.03 32.385 0)
+			(at 113.03 31.7499 0)
 			(effects
 				(font
@@
 			)
 		)
-		(property "Value" "100nF"
-			(at 113.03 34.925 0)
+		(property "Value" "0.1uF"
+			(at 113.03 34.2899 0)
 			(effects
 				(font
